Commit message: Changes in joints declaration

File: urdf/robot.urdf (robot description, URDF)
Before this commit: robot platform, 1 links, 2 joints
Joints:
- added joint axis_to_base_3: type fixed, parent base, child axis_base_21, origin xyz=0 0 0 rpy=0 0 0
- added joint axis_to_base_4: type fixed, parent base, child axis_base_22, origin xyz=0 0 0 rpy=0 0 0
- joint axis_to_base_1: child axis_1 -> axis_base_11
- joint axis_to_base_2: child axis_2 -> axis_base_12

Commit message: Added teleoperator control for robot

File: urdf/robot.urdf (robot description, URDF)
Before this commit: robot platform, 1 links, 4 joints
Links:
- added link dummy
Joints:
- added joint dummy_joint: type fixed, parent dummy, child base
